File: hardware/cowells_DUE_adapter_board/cowells_DUE_adapter_board.sch (KiCad schematic (older format))
At the start: 30 parts, among them J1 DRV8305J1, J2 DRV8305J1, J3 AS5048A, J4 AS5311AB, J5 AS5311AB, J6 AS5311AB, SW1 Run, SW2 Dir, SW3 eStop, SW4 sw_rst, SW5 SW_DIP_x03, U1 NL17SZ14, Y1 20MHz

Commit message: implemented current reading
current reading updated
Parts:
- removed R1, R2, R3: 10k, Resistors_SMD:R_0805_HandSoldering, symbol R
- added C? (x3): 15n, Capacitors_SMD:C_0805_HandSoldering, symbol C
- C1, C2: value Cm -> 18p
- J2: value DRV8305J1 -> DRV8305J2; footprint Pin_Headers:Pin_Header_Straight_1x08_Pitch2.54mm -> Pin_Headers:Pin_Header_Straight_2x10_Pitch2.54mm
- J4: value AS5311AB -> spindl enc.
- XA1: footprint Arduino:Arduino_Due_Shield -> Arduino:Arduino_Due_Shield_noHoles
- spd1: value 0.3k -> 5k
Connections:
- net CsnSpn: now also J4.5 (Pin_5); no longer J4.7 (Pin_7)
- net CsnX: now also J5.5 (Pin_5); no longer J5.7 (Pin_7)
- net CsnZ: now also J6.5 (Pin_5); no longer J6.7 (Pin_7)
- net GND: now also J4.6 (Pin_6), J5.6 (Pin_6), J6.6 (Pin_6), SW1.2 (B), SW2.2 (B), SW3.2 (B), XA1.GND2 (GND), XA1.GND3 (GND), XA1.GND5 (GND), XA1.GND6 (GND), C?.1, C?.1, C?.1
- net InH_A: now also XA1.D6; no longer XA1.D5
- net InH_B: now also XA1.D7; no longer XA1.D6
- net InH_C: now also XA1.D8; no longer XA1.D7
- net IsenA: now also XA1.A2; no longer XA1.A0
- net IsenC: now also XA1.A0; no longer XA1.A2
- net SCLK: no longer J5.6 (Pin_6), J6.6 (Pin_6)
- net VCC: no longer SW1.2 (B), SW2.2 (B), SW3.2 (B)
- net VsenA: now also SW5.4, XA1.A6; no longer SW5.6, XA1.A4
- net VsenC: now also SW5.6, XA1.A4; no longer SW5.4, XA1.A6
- net at SW1.1 (A), XA1.D23: now also C?.2
- net at SW2.1 (A), XA1.D25: now also C?.2
- net at SW3.1 (A), XA1.D27: now also C?.2
- net at J1.5 (Pin_5): now also SW5.3; no longer SW5.1
- net at J1.9 (Pin_9): now also SW5.1; no longer SW5.3
- net DoX renamed PWMx
- net PWMx: now also J5.7 (Pin_7); no longer J5.5 (Pin_5)
- net DoZ renamed PWMz
- net PWMz: now also J6.7 (Pin_7); no longer J6.5 (Pin_5)
- no-connect marks 85 -> 80
Other:
- note added: "Use with Input_Pullup"
- moved on the sheet: J4, SW1A, SW2A, SW3A
